Commit message: updated urdf code

File: urdf_tutorial-ros2/urdf/trevor.urdf (robot description, URDF)
Before this commit: robot trevor, 1 links, 0 joints
Links:
- added link frame; visual mesh filename=package://urdf_tutorial/meshes/frame.dae
- added link thrusters; visual mesh filename=package://urdf_tutorial/meshes/thruster.dae
Joints:
- added joint box_to_frame: type fixed, parent base_link, child frame, origin xyz=0 0 0
- added joint frame_to_thrusters: type fixed, parent frame, child thrusters, origin xyz=0 0 0
