Commit message: finished configuration

File: trevor_urdf/urdf/trevor.urdf (robot description, URDF)
Before this commit: robot trevor, 4 links, 3 joints
Links:
- link base_link: geometry visual mesh filename=package://trevor_urdf/meshes/usv_box.dae
- link frame: geometry visual mesh filename=package://trevor_urdf/meshes/frame.dae
- link thrusters: geometry visual mesh filename=package://trevor_urdf/meshes/thruster.dae

Commit message: URDF Changes

File: trevor_urdf/urdf/trevor.urdf (robot description, URDF)
Before this commit: robot trevor, 4 links, 3 joints
Links:
- link base_link: geometry 
- link frame: geometry visual mesh filename=package://trevor_urdf/meshes/full_usv.dae
